File: Hardware/Interconnect-Board/Interconnect-Board.kicad_pcb (KiCad board)
At the start: 2 copper layers, 32 x 47 mm, 6 parts, among them J1 Disp_Connector, J2 HMI_Daughter_Connector

Commit message: Bump kicad
Other:
- board text added: "${FULL_REVISION}"
- board text added: "JLCJLCJLCJLC"
Changed lines of the file:
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@@
+		)
+	)
+	(gr_text "${FULL_REVISION}"
+		(at -21.5 16 90)
+		(layer "F.SilkS")
+		(effects
+			(font
+				(size 0.9 0.9)
+				(thickness 0.18)
+				(bold yes)
+			)
+			(justify left top)
+		)
+	)
+	(gr_text "JLCJLCJLCJLC"
+		(at -19.5 16 90)
+		(layer "F.SilkS")
+		(effects
+			(font
+				(size 0.9 0.9)
+				(thickness 0.18)
+				(bold yes)
+			)
+			(justify left top)
 		)
 	)

Commit message: Add aux
Parts:
- added J3: AUX1, Connector_JST:JST_EH_B2B-EH-A_1x02_P2.50mm_Vertical, F.Cu at (-20.1, -12.9)
- added J4: AUX2, Connector_JST:JST_EH_B2B-EH-A_1x02_P2.50mm_Vertical, F.Cu at (-20.1, -3.54)
Connections:
- J2 pad 7: unconnected-(J2-Pin_7-Pad7) -> /AUX1
- J2 pad 9: unconnected-(J2-Pin_9-Pad9) -> /AUX2
Routing:
- net /AUX1: track 0.00 -> 13.1 mm
- net /AUX2: track 0.00 -> 9.16 mm
