File: Hardware/Interconnect-Board/Interconnect-Board.kicad_sch (KiCad schematic)
At the start: 2 parts, among them J1 Disp_Connector, J2 HMI_Daughter_Connector

Commit message: Move interconnect board
Other:
- title: EG-498-Temperature-Chamber-Team-Thermocline -> Interconnect-Board
Changed lines of the file:
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@@
 	(paper "A4")
 	(title_block
-		(title "EG-498-Temperature-Chamber-Team-Thermocline")
+		(title "Interconnect-Board")
 		(rev "${REVISION}")
 		(company "SNHU EG-498")
@@
 		)
 		(instances
-			(project "EG-498-Temperature-Chamber-Team-Thermocline"
+			(project "Interconnect-Board"
 				(path "/894f620e-3404-4a40-a2a7-513bc1d5f99b"
 					(reference "#PWR04")
@@
 		)
 		(instances
-			(project "EG-498-Temperature-Chamber-Team-Thermocline"
+			(project "Interconnect-Board"
 				(path "/894f620e-3404-4a40-a2a7-513bc1d5f99b"
 					(reference "#PWR06")

Commit message: Add aux
Parts:
- added J3: AUX1, Connector_JST:JST_EH_B2B-EH-A_1x02_P2.50mm_Vertical, symbol Connector_Generic:Conn_01x02
- added J4: AUX2, Connector_JST:JST_EH_B2B-EH-A_1x02_P2.50mm_Vertical, symbol Connector_Generic:Conn_01x02
Connections:
- net GND: now also J3.1 (Pin_1), J4.1 (Pin_1)
- net AUX1: now reaches J2.7 (Pin_7)
- net AUX1: now also J3.2 (Pin_2)
- net AUX2: now reaches J2.9 (Pin_9)
- net AUX2: now also J4.2 (Pin_2)
- no-connect marks 4 -> 2
